File: board/bench_pwr_rig/buck_boost.sch (KiCad schematic (older format))
At the start: 1 part

Commit message: Use photon
Updated schematic to use particle photon device for 3.3V interface to existing NHD-0208AZ-RN-YBW-3V in stock
Changed lines of the file:
@@
 EELAYER 29 0
 EELAYER END
-$Descr A4 11693 8268
+$Descr A3 16535 11693
 encoding utf-8
 Sheet 2 2
@@
 L Regulator_Switching:LM5176PWP U?
 U 1 1 5F8B8B75
-P 5400 3250
-F 0 "U?" H 5400 4431 50  0000 C CNN
-F 1 "LM5176PWP" H 5400 4340 50  0000 C CNN
-F 2 "Package_SO:HTSSOP-28-1EP_4.4x9.7mm_P0.65mm_EP3.4x9.5mm_ThermalVias" H 6100 4100 50  0001 L CNN
-F 3 "http://www.ti.com/lit/ds/symlink/lm5176.pdf" H 7400 2800 50  0001 C CNN
-	1    5400 3250
+P 4950 8350
+F 0 "U?" H 4950 9531 50  0000 C CNN
+F 1 "LM5176PWP" H 4950 9440 50  0000 C CNN
+F 2 "Package_SO:HTSSOP-28-1EP_4.4x9.7mm_P0.65mm_EP3.4x9.5mm_ThermalVias" H 5650 9200 50  0001 L CNN
+F 3 "http://www.ti.com/lit/ds/symlink/lm5176.pdf" H 6950 7900 50  0001 C CNN
+	1    4950 8350
 	1    0    0    -1
 $EndComp

Commit message: Updated powertrain schematic
Changed powertrain to PSFB
Updated schematic
Added new symbols
Parts:
- removed U?: LM5176PWP, Package_SO:HTSSOP-28-1EP_4.4x9.7mm_P0.65mm_EP3.4x9.5mm_ThermalVias, symbol Regulator_Switching:LM5176PWP
- added C? (x10): C, symbol Device:C
- added C? (x2): C_Polarized, symbol Device:C_Polarized
- added D?: 1N4148W, Diode_SMD:D_SOD-123, symbol Diode:1N4148W
- added D? (x4): MURS360T3G, Diode_SMD:D_SMC_Handsoldering, symbol Diode:MURS360T3G
- added D? (x8): BAT54W, Package_TO_SOT_SMD:SOT-323_SC-70, symbol Diode:BAT54W
- added D? (x2): BAT42W-V, Diode_SMD:D_SOD-123, symbol Diode:BAT42W-V
- added F?: Fuse, symbol Device:Fuse
- added L?: SER1512-103, symbol Inductor:SER1512-103
- added Q? (x4): STF26N60M2, Package_TO_SOT_THT:TO-220-3_Vertical, symbol Transistor_FET:STF26N60M2
- added Q? (x4): STP110N10F7, Package_TO_SOT_THT:TO-220-3_Vertical, symbol Transistor_FET:STP110N10F7
- added R? (x29): R, symbol Device:R
- added T?: CST1211, symbol Transformer:CST1211
- added U?: UCC28951, Package_SO:TSSOP-24_4.4x7.8mm_P0.65mm, symbol Regulator_Controller:UCC28951
- added U? (x4): UCC27714D, Package_SO:SOIC-14_3.9x8.7mm_P1.27mm, symbol Driver_FET:UCC27714D
- added U?: AGP2923-333, symbol Inductor:AGP2923-333
- added U? (x3): TLC272, symbol Amplifier_Operational:TLC272
- added U?: ISO7240MDW, Package_SO:SOIC-16W_7.5x10.3mm_P1.27mm, symbol Isolator:ISO7240MDW
Connections:
- net labels added: AO, BO, CO, DO, GNDA, GNDREF, OUTA, OUTB, OUTC, OUTE, OUTF, SWAB, SWCD, Vdrive
- wire segments 0 -> 248
- no-connect marks 0 -> 4
