File: board/bench_pwr_rig/PSFB.sch (KiCad schematic (older format))
At the start: 127 parts

Commit message: Schematic Update
Updated schematic
Added Input Filter and PFC sections
Added capacitor, resistor, and protection parts library
Started a jupyter notebook for PFC section
Parts:
- removed C? (x13): C, symbol Device:C
- removed C? (x2): C_Polarized, symbol Device:C_Polarized
- removed R? (x33): R, symbol Device:R
- added C? (x4): EEU-EB1J221, Capacitor_THT:CP_Radial_D10.0mm_P5.00mm, symbol Capacitor:EEU-EB1J221
- added C?: C4AEHBU5100A11J, Capacitor_THT:C_Rect_L33.0mm_W20.0mm_P27.50mm_MKS4, symbol Capacitor:C4AEHBU5100A11J
- added C? (x8): C1608X7R1H104K, Capacitor_SMD:C_0603_1608Metric_Pad1.05x0.95mm_HandSolder, symbol Capacitor:C1608X7R1H104K
- added C? (x3): C, symbol Device:C
- added C? (x9): C1608X7R1E105K080AB, Capacitor_SMD:C_0603_1608Metric_Pad1.05x0.95mm_HandSolder, symbol Capacitor:C1608X7R1E105K080AB
- added D? (x2): BAS316, Diode_SMD:D_SOD-323, symbol Diode:BAS316
- added D?: 19-217_GHC-YR1S2_3T, LED_SMD:LED_0603_1608Metric_Pad1.05x0.95mm_HandSolder, symbol LED:19-217_GHC-YR1S2_3T
- added R?: 0603WAF1001T5E, Resistor_SMD:R_0603_1608Metric_Pad1.05x0.95mm_HandSolder, symbol Resistor:0603WAF1001T5E
- added R?: 0603WAF4871T5E, Resistor_SMD:R_0603_1608Metric_Pad1.05x0.95mm_HandSolder, symbol Resistor:0603WAF4871T5E
- added R? (x5): R, symbol Device:R
- added R? (x9): CRCW060310K0FKEA, Resistor_SMD:R_0603_1608Metric_Pad1.05x0.95mm_HandSolder, symbol Resistor:CRCW060310K0FKEA
- added R? (x12): CRCW08052R21FKEA, Resistor_SMD:R_0805_2012Metric_Pad1.15x1.40mm_HandSolder, symbol Resistor:CRCW08052R21FKEA
- added R? (x4): 0603WAF5111T5E, Resistor_SMD:R_0603_1608Metric_Pad1.05x0.95mm_HandSolder, symbol Resistor:0603WAF5111T5E
- added R? (x4): 0603WAF7151T5E, Resistor_SMD:R_0603_1608Metric_Pad1.05x0.95mm_HandSolder, symbol Resistor:0603WAF7151T5E
- added R? (x2): 0603WAF8251T5E, Resistor_SMD:R_0603_1608Metric_Pad1.05x0.95mm_HandSolder, symbol Resistor:0603WAF8251T5E
- added R?: 0603WAF8253T5E, Resistor_SMD:R_0603_1608Metric_Pad1.05x0.95mm_HandSolder, symbol Resistor:0603WAF8253T5E
- added R?: 0603WAF226JT5E, Resistor_SMD:R_0603_1608Metric_Pad1.05x0.95mm_HandSolder, symbol Resistor:0603WAF226JT5E
- added R?: CRCW0603221RFKEA, Resistor_SMD:R_0603_1608Metric_Pad1.05x0.95mm_HandSolder, symbol Resistor:CRCW0603221RFKEA
- added T?: PQ2625_PROTO, Transformer_THT:CPV-PQ26-25-1S-12PD-Z, symbol Transformer:PQ2625_PROTO
- added U?: LM78L05_TO92, Package_TO_SOT_THT:TO-92_Inline, symbol Regulator_Linear:LM78L05_TO92
- added U?: OPA376xxDBV, Package_TO_SOT_SMD:SOT-23-5, symbol Amplifier_Operational:OPA376xxDBV
- T?: footprint (none) -> Transformer_SMD:Transformer_Coilcraft_CST1211
- U?: footprint (none) -> Inductor_THT:L_Coilcraft_AGP2923
Connections:
- net GNDREF is gone; now on net GND: C?.2
- net VOUT is gone; now on net OUTP: C?.1, R?.1, U?.2
- net +5V: now also C?.1, C?.1, C?.2, U?.5 (V+)
- net GND: now also C?.2, R?.2, R?.2, T?.4, C?.1, C?.1, C?.1, C?.1, C?.1, C?.1, C?.1, C?.2, C?.2, C?.2, C?.2, C?.2, C?.2, C?.2, C?.2, C?.2, C?.2, C?.2, C?.2, D?.1 (K), R?.1, R?.1, R?.2, R?.2, R?.2, R?.2, R?.2, R?.2, R?.2, R?.2, R?.2, R?.2, R?.2, U?.2 (GND), U?.2 (V-)
- net IO_SNS: now also C?.1, R?.1, U?.1
- net OUTA: now also R?.1
- net OUTB: now also R?.1
- net OUTC: now also R?.1, R?.1
- net OUTE: now also U?.1 (HI), U?.2 (LI); no longer U?.1 (HI), U?.2 (LI)
- net OUTF: now also U?.1 (HI), U?.2 (LI); no longer U?.1 (HI), U?.2 (LI)
- net OUTN: now also R?.1, R?.1
- net OUTP: now also C?.1, C?.1, C?.1, C?.1
- net SWAB: now also T?.1, T?.2, T?.3
- net SWCD: now also C?.2, R?.2, T?.4, T?.5, T?.6
- net VREF: now also C?.2, R?.1, R?.1, R?.1
- net at Q?.1 (G): now also R?.1, R?.1 (x4)
- net at D?.3 (K), U?.12 (HO): now also R?.2 (x2)
- net at D?.1 (A), L?.1, Q?.2 (D)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: now also C?.2, R?.2
- net at D?.3 (K), U?.6 (LO): now also R?.2 (x2)
- net at F?.1, T?.1: now also C?.1
- net at R?.1, U?.13 (ADELEF): now also R?.2
- net at R?.1, U?.14 (ADEL): now also R?.2
- net at C?.1, R?.1, U?.15 (CS): now also R?.1
- net at D?.2 (A), D?.2 (A), U?.2 (EA+): now also R?.2
- net at U?.23 (VDD): now also C?.2, C?.2, R?.2
- net at C?.1, U?.5 (SS/EN): now also R?.1
- net at Q?.1 (G): now also R?.1, R?.2 (x4)
- net SWF: now reaches D?.1 (A), Q?.2 (D), Q?.3 (S), U?.11 (HS)
- net SWF: now also C?.2, R?.2, T?.10, T?.11, T?.12
- net SWE: now reaches D?.1 (A), Q?.2 (D), Q?.3 (S), U?.11 (HS)
- net SWE: now also C?.2, R?.2, T?.7, T?.8, T?.9
- net at D?.1 (K), U?.13 (HB): now also C?.1 (x2)
- net at D?.3 (K), U?.12 (HO): now also R?.1 (x2)
- net at D?.3 (K), U?.6 (LO): now also R?.1 (x2)
- net at D?.2 (A), T?.5: now also R?.1
- net at D?.1 (K), R?.1: now also R?.2
- net at D?.2 (A): now also R?.1
- net at U?.13 (HB): now also C?.1, D?.1 (K) (x2)
- net at D?.2 (A): now also R?.2
- net +5VP: now reaches U?.10 (EN), U?.16 (VCC2)
- net +5VP: now also C?.1, C?.1, R?.1, U?.1 (VO)
- net at U?.3 (INA): now also R?.1, R?.2
- net at U?.4 (INB): now also R?.1, R?.2
- net at U?.5 (INC): now also R?.1, R?.2
- net at U?.6 (IND): now also R?.1, R?.2
- net +10V renamed +12V
- net +12V: now also C?.1, C?.2, R?.1, R?.1, R?.2
- net Vdrive renamed VBIASP
- net VBIASP: now also C?.1, C?.1, C?.2, R?.1, R?.2, U?.3 (VI)
- new net: C?.1, C?.2, R?.2, R?.2, U?.3 (+)
- new net: C?.2, C?.2, R?.2, R?.2, U?.4 (-)
- new net: D?.2 (A), R?.1
- new net: D?.2 (A), R?.2 (x2)
Other:
- moved on the sheet: C?, D?, Q?, R?, U?, U?A, U?B, U?C

Commit message: schematic and layout updates
Finalized schematic for rev 0.1. Anticipate additional component values update through analysis. Moving to layout
Parts:
- removed C? (x13): C, symbol Device:C
- removed C?: C1608X7R1H104K, Capacitor_SMD:C_0603_1608Metric_Pad1.05x0.95mm_HandSolder, symbol Capacitor:C1608X7R1H104K
- removed D? (x8): BAT54W, Package_TO_SOT_SMD:SOT-323_SC-70, symbol Diode:BAT54W
- removed D? (x2): BAS316, Diode_SMD:D_SOD-323, symbol Diode:BAS316
- removed F?: Fuse, symbol Device:Fuse
- removed R? (x34): R, symbol Device:R
- removed R? (x8): CRCW08052R21FKEA, Resistor_SMD:R_0805_2012Metric_Pad1.15x1.40mm_HandSolder, symbol Resistor:CRCW08052R21FKEA
- removed T?: PQ2625_PROTO, Transformer_THT:CPV-PQ26-25-1S-12PD-Z, symbol Transformer:PQ2625_PROTO
- added C17, C34, C47: C1608C0G1H272J, Capacitor_SMD:C_0603_1608Metric_Pad1.05x0.95mm_HandSolder, symbol Capacitor:C1608C0G1H272J
- added C22: CL10C331JB8NNNC, Capacitor_SMD:C_0603_1608Metric_Pad1.05x0.95mm_HandSolder, symbol Capacitor:CL10C331JB8NNNC
- added C29: CL10B154KA8NNNC, Capacitor_SMD:C_0603_1608Metric_Pad1.05x0.95mm_HandSolder, symbol Capacitor:CL10B154KA8NNNC
- added C30: C1608X7R1E105K080AB, Capacitor_SMD:C_0603_1608Metric_Pad1.05x0.95mm_HandSolder, symbol Capacitor:C1608X7R1E105K080AB
- added C31, C48, C49: CL10B223KB8NNNC, Capacitor_SMD:C_0603_1608Metric_Pad1.05x0.95mm_HandSolder, symbol Capacitor:CL10B223KB8NNNC
- added C32, C35, C38: C1608X7R1H104K, Capacitor_SMD:C_0603_1608Metric_Pad1.05x0.95mm_HandSolder, symbol Capacitor:C1608X7R1H104K
- added C33: C1608C0G1H561J, Capacitor_SMD:C_0603_1608Metric_Pad1.05x0.95mm_HandSolder, symbol Capacitor:C1608C0G1H561J
- added C36, C39: DNP, Capacitor_SMD:C_0603_1608Metric_Pad1.05x0.95mm_HandSolder, symbol Capacitor:DNP
- added D10: 19-217_GHC-YR1S2_3T, LED_SMD:LED_0603_1608Metric_Pad1.05x0.95mm_HandSolder, symbol LED:19-217_GHC-YR1S2_3T
- added D12, D13, D16, D17, D20, D21, D6, D7: BAT54J, Diode_SMD:D_SOD-323F, symbol Diode:BAT54J
- added D15, D22: US1B, Diode_SMD:D_SMA, symbol Diode:US1B
- added Q10, Q13, Q14: BSS138, Package_TO_SOT_SMD:SOT-23, symbol Transistor_FET:BSS138
- added Q5: MMBT3906, Package_TO_SOT_SMD:SOT-23, symbol Transistor_BJT:MMBT3906
- added R100, R56, R98: 0603WAF1001T5E, Resistor_SMD:R_0603_1608Metric_Pad1.05x0.95mm_HandSolder, symbol Resistor:0603WAF1001T5E
- added R101, R102: 0603WAF1653T5E, Resistor_SMD:R_0603_1608Metric_Pad1.05x0.95mm_HandSolder, symbol Resistor:0603WAF1653T5E
- added R20: 1206W4F6983T5E, Resistor_SMD:R_1206_3216Metric_Pad1.42x1.75mm_HandSolder, symbol Resistor:1206W4F6983T5E
- added R21, R24: 1206W4F7153T5E, Resistor_SMD:R_1206_3216Metric_Pad1.42x1.75mm_HandSolder, symbol Resistor:1206W4F7153T5E
- added R22, R23, R41, R42, R68, R69, R90, R91: 0603WAF220KT5E, Resistor_SMD:R_0603_1608Metric_Pad1.05x0.95mm_HandSolder, symbol Resistor:0603WAF220KT5E
- added R25: 0603WAF6811T5E, Resistor_SMD:R_0603_1608Metric_Pad1.05x0.95mm_HandSolder, symbol Resistor:0603WAF6811T5E
- added R28: 0603WAF9093T5E, Resistor_SMD:R_0603_1608Metric_Pad1.05x0.95mm_HandSolder, symbol Resistor:0603WAF9093T5E
- added R29: 0603WAF4752T5E, Resistor_SMD:R_0603_1608Metric_Pad1.05x0.95mm_HandSolder, symbol Resistor:0603WAF4752T5E
- added R30: 0603WAF1003T5E, Resistor_SMD:R_0603_1608Metric_Pad1.05x0.95mm_HandSolder, symbol Resistor:0603WAF1003T5E
- added R31: 0603WAF8251T5E, Resistor_SMD:R_0603_1608Metric_Pad1.05x0.95mm_HandSolder, symbol Resistor:0603WAF8251T5E
- added R34, R72, R74, R75, R76: CRCW060310K0FKEA, Resistor_SMD:R_0603_1608Metric_Pad1.05x0.95mm_HandSolder, symbol Resistor:CRCW060310K0FKEA
- added R37, R96, R97: 0603WAF4872T5E, Resistor_SMD:R_0603_1608Metric_Pad1.05x0.95mm_HandSolder, symbol Resistor:0603WAF4872T5E
- added R50: 0603WAF3480T5E, Resistor_SMD:R_0603_1608Metric_Pad1.05x0.95mm_HandSolder, symbol Resistor:0603WAF3480T5E
- added R51, R57, R60, R80, R85: DNP, Resistor_SMD:R_0603_1608Metric_Pad1.05x0.95mm_HandSolder, symbol Resistor:DNP
- added R53: 0603WAF4221T5E, Resistor_SMD:R_0603_1608Metric_Pad1.05x0.95mm_HandSolder, symbol Resistor:0603WAF4221T5E
- added R55: 0603WAF1692T5E, Resistor_SMD:R_0603_1608Metric_Pad1.05x0.95mm_HandSolder, symbol Resistor:0603WAF1692T5E
- added R58: 0603WAF1273T5E, Resistor_SMD:R_0603_1608Metric_Pad1.05x0.95mm_HandSolder, symbol Resistor:0603WAF1273T5E
- added R59: 0603WAF6192T5E, Resistor_SMD:R_0603_1608Metric_Pad1.05x0.95mm_HandSolder, symbol Resistor:0603WAF6192T5E
- added R61: CRCW060313K0FKEA, Resistor_SMD:R_0603_1608Metric_Pad1.05x0.95mm_HandSolder, symbol Resistor:CRCW060313K0FKEA
- added R63: 0603WAF1402T5E, Resistor_SMD:R_0603_1608Metric_Pad1.05x0.95mm_HandSolder, symbol Resistor:0603WAF1402T5E
- added R64, R65: 0603WAF3012T5E, Resistor_SMD:R_0603_1608Metric_Pad1.05x0.95mm_HandSolder, symbol Resistor:0603WAF3012T5E
- added R73, R79: 0603WAF226JT5E, Resistor_SMD:R_0603_1608Metric_Pad1.05x0.95mm_HandSolder, symbol Resistor:0603WAF226JT5E
- added R77: 0603WAF1503T5E, Resistor_SMD:R_0603_1608Metric_Pad1.05x0.95mm_HandSolder, symbol Resistor:0603WAF1503T5E
- added R78: 0603WAF6812T5E, Resistor_SMD:R_0603_1608Metric_Pad1.05x0.95mm_HandSolder, symbol Resistor:0603WAF6812T5E
- added R81, R84: 0603WAF9092T5E, Resistor_SMD:R_0603_1608Metric_Pad1.05x0.95mm_HandSolder, symbol Resistor:0603WAF9092T5E
- added R83, R92, R93, R95: 0603WAF2491T5E, Resistor_SMD:R_0603_1608Metric_Pad1.05x0.95mm_HandSolder, symbol Resistor:0603WAF2491T5E
- added R88: 0603WAF2802T5E, Resistor_SMD:R_0603_1608Metric_Pad1.05x0.95mm_HandSolder, symbol Resistor:0603WAF2802T5E
- added R89: CRCW060333K2FKEA, Resistor_SMD:R_0603_1608Metric_Pad1.05x0.95mm_HandSolder, symbol Resistor:CRCW060333K2FKEA
- added R99: CSS4J-4026R-L500, Resistor_SMD:R_Shunt_Bourns_CSS4J_4026, symbol Resistor:CSS4J-4026R-L500
- added T2: PQ2625_PROTO, Transformer_THT:CPV-PQ26-25-1S-12PD-Z, symbol Transformer:PQ2625_PROTO
- added U10: TL431DBZ, Package_TO_SOT_SMD:SOT-23, symbol Reference_Voltage:TL431DBZ
- added U11: FODM217B, Package_SO:SOP-4_4.4x2.6mm_P1.27mm, symbol Isolator:FODM217B
- C19, C37, C41: renamed from C?; value C -> DNP; footprint (none) -> Capacitor_SMD:C_1206_3216Metric
- L1: renamed from L?; footprint (none) -> Inductor_SMD:L_Coilcraft_SER1512
- Q6, Q7, Q8, Q9: renamed from Q?; footprint Package_TO_SOT_THT:TO-220-3_Vertical -> Package_TO_SOT_THT:TO-220-3_Vertical_Stag
- R82: renamed from R?; value R -> DNP; footprint (none) -> Resistor_SMD:R_1206_3216Metric
- U16: renamed from U?; footprint (none) -> Package_SO:SOIC-8_3.9x4.9mm_P1.27mm
- gave numbers to parts that had none: 72
Connections:
- net +5V: now also C30.1, R34.1, R74.1
- net GND: now also T1.5, C22.2, C29.2, C30.2, C35.1, C38.1, C48.1, D16.2 (A), D21.2 (A), Q10.2 (S), Q13.2 (S), Q14.2 (S), R102.1, R37.2, R50.2, R51.2, R53.2, R56.2, R58.2, R60.2, R61.2, R63.2, R64.2, R65.2, R72.2, R75.2, R76.2, R81.1, R83.2, R84.1, R99.4, U11.3; no longer C12.2, C13.2, C14.2, C16.2, C18.2, C19.2, C23.1, D4.1 (K), D9.2 (A), Q7.3 (S), Q9.3 (S), R27.2, R39.2, T1.4, U12.15 (GND2), U12.9 (GND2), U13.3 (VSS), U13.5 (COM), U8.2 (GND), U9.3 (VSS), U9.5 (COM)
- net ICTL: now also R92.1
- net IO_SNS: now also C49.2, R101.1, R96.1
- net OUTC: no longer R46.1, U14.19 (OUTD)
- net OUTN: now also R99.1
- net OUTP: now also R97.1
- net SWAB: now also T2.1, T2.2, T2.3
- net SWCD: now also D12.2 (A), T2.4, T2.5, T2.6
- net SWE: now also D20.2 (A), T2.7, T2.8, T2.9
- net SWF: now also D17.2 (A), T2.10, T2.11, T2.12
- net VBIASP: now also D10.2 (A), Q5.2 (E), R29.1
- net VCTL: now also R93.1
- net VINP: now also C16.1, T1.2, R20.2
- net VREF: now also R55.1, R57.1, R59.1
- net RT: now reaches U14.10 (RT)
- net RT: now also R59.2, R60.1
- net RSUM: now reaches U14.11 (RSUM)
- net RSUM: now also R57.2, R58.1
- net DCM: now reaches U14.12 (DCM)
- net DCM: now also R55.2, R56.1
- net ADELEF: now reaches R52.2, U14.13 (ADELEF)
- net ADELEF: now also R53.1
- net ADEL: now reaches R49.2, U14.14 (ADEL)
- net ADEL: now also R50.1
- net CS: now reaches R47.1, U14.15 (CS)
- net CS: now also C22.1, R51.1
- net EA+: now reaches D18.2 (A), D19.2 (A), R62.2, U14.2 (EA+)
- net U14-VDD: now reaches C24.2, C25.2, R54.2, U14.23 (VDD)
- net COMP: now reaches U14.3 (EA-), U14.4 (COMP)
- net SS-EN: now reaches R67.1, U14.5 (SS/EN)
- net SS-EN: now also C29.1, Q10.3 (D), Q13.3 (D)
- net DELAB: now reaches U14.6 (DELAB)
- net DELAB: now also R65.1
- net DELCD: now reaches U14.7 (DELCD)
- net DELCD: now also R64.1
- net DELEF: now reaches U14.8 (DELEF)
- net DELEF: now also R63.1
- net TMIN: now reaches U14.9 (TMIN)
- net TMIN: now also R61.1
- net Q6-G: now reaches Q6.1 (G), R26.1
- net Q6-G: now also R23.1
- net VINX: now reaches D8.1 (K), Q6.2 (D), Q8.2 (D)
- net VINX: now also T1.1; no longer T1.2
- net U9-HS: now reaches C15.2, L1.1, Q6.3 (S), Q7.2 (D), R26.2, U9.11 (HS)
- net U9-HS: now also D7.2 (A)
- net Q7-G: now reaches Q7.1 (G), R27.1
- net Q7-G: now also R22.1
- net Q8-G: now reaches Q8.1 (G), R38.1
- net Q8-G: now also R41.2
- net Q9-G: now reaches Q9.1 (G), R39.1
- net Q9-G: now also R42.2
- net at Q11.1 (G), R70.1: now also R68.1
- net Q15-G: now reaches Q15.1 (G), R86.1
- net Q15-G: now also R90.2
- net Q12-G: now reaches Q12.1 (G), R71.1
- net Q12-G: now also R69.1
- net at Q16.1 (G), R87.1: now also R91.2
- net U9-HO: now reaches U9.12 (HO)
- net U9-HO: now also D7.1 (K), R23.2
- net U9-HB: now reaches C15.1, D5.1 (K), U9.13 (HB)
- net U9-LO: now reaches U9.6 (LO)
- net U9-LO: now also D6.1 (K), R22.2
- net U13-HO: now reaches U13.12 (HO)
- net U13-HO: now also D12.1 (K), R41.1
- net U13-HB: now reaches C21.1, D14.1 (K), U13.13 (HB)
- net U13-LO: now reaches U13.6 (LO)
- net U13-LO: now also D13.1 (K), R42.1
- net CS-P: now reaches D11.2 (A), R33.1
- net CS-P: now also T1.4; no longer T1.5
- net CS-RECT: now reaches D11.1 (K), R47.2
- net CS-RECT: now also R37.1
- net U15-HO: now reaches U15.12 (HO)
- net U15-HO: now also D17.1 (K), R68.2
- net U15-HB: now reaches C28.1, U15.13 (HB)
- net U15-HB: now also D15.1 (K)
- net U15-LO: now reaches U15.6 (LO)
- net U15-LO: now also D16.1 (K), R69.2
- net U18-HO: now reaches U18.12 (HO)
- net U18-HO: now also D20.1 (K), R90.1
- net U18-HB: now reaches C40.1, U18.13 (HB)
- net U18-HB: now also D22.1 (K)
- net U18-LO: now reaches U18.6 (LO)
- net U18-LO: now also D21.1 (K), R91.1
- net at D19.1 (K), U16.1: now also C32.2, C34.2
- net at U16.2 (-): now also C34.1, R78.1, R83.1, R85.2, R89.2
- net at U16.3 (+): now also C38.2, R84.2, R93.2
- net at U16.5 (+): now also C35.2, R81.2, R92.2
- net at U16.6 (-): now also C33.1, R77.1, R80.2, R88.2
- net at D18.1 (K), U16.7: now also C31.2, C33.2
- net at U19.3 (+): now also C47.1, C48.2, R100.2, R102.2
- net at U19.4 (-): now also C47.2, C49.1, R101.2, R98.2
- net at R66.1: now also D15.2 (A)
- net at R94.2: now also D22.2 (A)
- new net: R100.1, R99.2
- new net: R98.1, R99.3
- new net: C39.1, R89.1, R95.2
- new net: C39.2, R85.1
- new net: C36.1, R88.1, R96.2
- new net: C36.2, R80.1
- new net: R95.1, R97.2
- new net: C32.1, R78.2
- new net: C31.1, R77.2
- new net: Q10.1 (G), R72.1, R73.2
- new net: R30.2, R31.2, U11.1
- new net: U10.1 (K), U11.2
- new net: Q13.1 (G), Q14.3 (D), R74.2, R75.1
- new net: Q14.1 (G), R76.1, R79.2
- new net: C17.1, R24.1, R25.1, R28.2, U10.2 (REF)
- new net: D10.1 (K), R31.1
- new net: R20.1, R21.2
- new net: R21.1, R24.2
- new net: Q5.3 (C), R28.1
- new net: Q5.1 (B), R29.2, R30.1
- new net OUTD: R46.1, U14.19 (OUTD)
- new net PSFB_ON: R79.1
- new net VINN: C12.2, C13.2, C14.2, C16.2, C17.2, C18.2, C19.2, C23.1, D13.2 (A), D4.1 (K), D6.2 (A), D9.2 (A), Q7.3 (S), Q9.3 (S), R25.2, R27.2, R39.2, U10.3 (A), U12.15 (GND2), U12.9 (GND2), U13.3 (VSS), U13.5 (COM), U8.2 (GND), U9.3 (VSS), U9.5 (COM)
- new net VIN_PG: R34.2, R73.1, U11.4
Other:
- moved on the sheet: C12, C14, C50, D4, R19, R67, U8
