File: board/bench_pwr_rig/bench_pwr_rig.kicad_pcb (KiCad board)
At the start: 2 copper layers, 259 parts, among them J1 703W-00_54, K1 G5Q-1A, Q1 Si2319CDS, Q10 BSS138, Q11 STP110N10F7, Q12 STP110N10F7, Q13 BSS138, Q14 BSS138, Q15 STP110N10F7, Q16 STP110N10F7, Q17 SCTW35N65G2V, Q2 BSS138, Q3 STP110N10F7, Q4 STP110N10F7, Q5 MMBT3906, Q6 STF26N60M2, Q7 STF26N60M2, Q8 STF26N60M2, Q9 STF26N60M2, SW1 SW_SPDT, T1 CST1211, T2 PQ2625_PROTO, T3 7448251201, T4 7448251201, U1 FODM217B, U10 TL431DBZ, U11 FODM217B, U12 ISO7240MDW, U13 UCC27714D, U14 UCC28951, U15 UCC27714D, U16 TLC272, U17 AGP2923-333, U18 UCC27714D, U19 OPA376xxDBV, U2 PEME1-S5-S12-S, U20 UCC28180D, U21 UCC27517DBV, U3 LM317_TO-220, U4 PBO-3-S12, U5 LTC4359-MS8, U6 PHOTON-MCU_Module, U7 NHD-0208AZ-RN-YBW-3V, U8 LM78L05_TO92, U9 UCC27714D

Commit message: Updated layout
Added output screw terminal
Added mounting screws M4
Changed primary ground to secondary ground plane coupling capacitor to radial disc type with safety rating X1, Y1
Continued layout
Parts:
- removed U17: AGP2923-333, Inductor_THT:L_Coilcraft_AGP2923
- added C59: C, Capacitor_THT:C_Disc_D9.0mm_W5.0mm_P10.00mm, F.Cu at (337.3, 100.1)
- added H1: MountingHole, MountingHole:MountingHole_4.3mm_M4, F.Cu at (78.7, 101.6)
- added H2: MountingHole, MountingHole:MountingHole_4.3mm_M4, F.Cu at (412.0, 101.6)
- added H3: MountingHole, MountingHole:MountingHole_4.3mm_M4, F.Cu at (78.7, 172.7)
- added H4: MountingHole, MountingHole:MountingHole_4.3mm_M4, F.Cu at (181.4, 101.6)
- added H5: MountingHole, MountingHole:MountingHole_4.3mm_M4, F.Cu at (412.0, 172.7)
- added H6: MountingHole, MountingHole:MountingHole_4.3mm_M4, F.Cu at (237.7, 172.7)
- added J2: Screw_Terminal_01x02, TerminalBlock_Phoenix:TerminalBlock_Phoenix_MKDS-1,5-2-5.08_1x02_P5.08mm_Horizontal, F.Cu at (411.0, 114.8)
- added J3: Screw_Terminal_01x02, TerminalBlock_Phoenix:TerminalBlock_Phoenix_MKDS-1,5-2-5.08_1x02_P5.08mm_Horizontal, F.Cu at (411.0, 140.2)
- added L3: AGP2923-333, Inductor_THT:L_Coilcraft_AGP2923, F.Cu at (378.5, 107.2)
- C11, C8, D15, R14, R66, R9, U5: moved to F.Cu
- C19: value DNP -> C; footprint Capacitor_SMD:C_1206_3216Metric -> Capacitor_THT:C_Disc_D9.0mm_W5.0mm_P10.00mm; moved to F.Cu
- C22, C37, C41, Q14, R115, R116, R13, R15, R17, R51, R74, R76, R79, R82, SW1: moved to B.Cu
- C57: value C1608X7R1H104K -> CC0805KRX7R9BB104; footprint Capacitor_SMD:C_0603_1608Metric_Pad1.05x0.95mm_HandSolder -> Capacitor_SMD:C_0805_2012Metric_Pad1.15x1.40mm_HandSolder
- C58: value C1608X7R1E105K080AB -> CL21B105KBFNNNE; footprint Capacitor_SMD:C_0603_1608Metric_Pad1.05x0.95mm_HandSolder -> Capacitor_SMD:C_0805_2012Metric_Pad1.15x1.40mm_HandSolder
- R75: value CRCW060310K0FKEA -> 0603WAF4752T5E
- moved R82 108.2 mm to (317.4, 84.6)
- moved C37 104.7 mm to (317.4, 87.6)
- moved SW1 49.3 mm to (415.0, 150.4), turned to 270 degrees
- moved C63 45.2 mm to (255.5, 106.7)
- moved R114 44.9 mm to (230.1, 155.4)
- moved R113 44.4 mm to (235.7, 155.4)
- moved R112 43.9 mm to (241.3, 155.4)
- moved C19 42.0 mm to (321.6, 100.1)
- moved C61 36.7 mm to (236.7, 145.3)
- moved R16 23.0 mm to (372.9, 172.7)
- moved R107 23.0 mm to (208.3, 117.3)
- moved R17 23.0 mm to (398.3, 162.6)
- moved R105 22.9 mm to (208.3, 122.4)
- moved R106 22.9 mm to (208.3, 127.5)
- moved C41 22.8 mm to (386.5, 128.5)
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Connections:
- net Net-(C11-Pad1) renamed /OUTP-DOR
- net Net-(C11-Pad2) renamed /U5-VSS
- net Net-(C51-Pad1) renamed /PFC/U20-ISNS
- net Net-(C52-Pad1) renamed /PFC/U20-ICOMP
- net Net-(C55-Pad1) renamed /PFC/BST-VCMP
- net Net-(C64-Pad2) renamed /Inputfilter/N_AC_FUSE
- net Net-(C65-Pad1) renamed /Inputfilter/L_AC_MID
- net Net-(C66-Pad2) renamed /Inputfilter/N_AC_MID
- net Net-(D2-Pad2) renamed /N_FILT_AC_RT
- net Net-(D25-Pad2) renamed /PFC/BST-SW-NODE
- net Net-(Q11-Pad2) renamed /PSFB/SW_LOUT
- net Net-(Q3-Pad3) renamed /OUTP-SWTCHD
- net Net-(Q4-Pad1) renamed /OUT-G-DRV
- net Net-(R104-Pad1) renamed /PFC/BST-FREQ
- net Net-(R111-Pad1) renamed /PFC/BST-VSNS
- net Net-(U20-Pad8) renamed /PFC/U20-OUT
- C19 pad 1: GND -> Net-(C19-Pad1)
- R10 pad 2: /IO_SNS -> /VO_SNS
- R74 pad 1: +5V -> /PSFB/VREF
- R9 pad 2: /VO_SNS -> /IO_SNS
- U6 pad 10: Net-(SW1-Pad2) -> Net-(C8-Pad1)
- U6 pad 11: Net-(C8-Pad1) -> Net-(R16-Pad2)
- U6 pad 12: Net-(C10-Pad1) -> /INRUSH_RELAY_EN
- U6 pad 19: Net-(R16-Pad2) -> Net-(SW1-Pad2)
- U6 pad 20: Net-(R15-Pad2) -> /OUT_EN
- U6 pad 6: /ICTL -> /VCTL
- U6 pad 7: /INRUSH_RELAY_EN -> Net-(R15-Pad2)
- U6 pad 8: /OUT_EN -> Net-(C10-Pad1)
- U6 pad 9: /VCTL -> /ICTL
Routing:
- net GND: track 93.7 -> 385.3 mm, vias 4 -> 8
- net +5V: track 84.0 -> 353.4 mm, vias 1 -> 6
- net +12V: track 95.9 -> 276.3 mm, vias 3 -> 6
- net /VBIASP: track 5.93 -> 134.5 mm, vias 1 -> 3
- net /INRUSH_RELAY_EN: track 111.6 -> 181.7 mm, vias 0 -> 1
- net /PFC_ON: track 106.5 -> 173.4 mm, vias 0 -> 2
- net +3V3: track 0.00 -> 63.3 mm, vias 0 -> 1
- net /RTNP: track 25.4 -> 86.3 mm, vias 0 -> 11
- net Net-(R15-Pad2): track 0.00 -> 60.2 mm, vias 0 -> 2
- net /PSFB/VINP: track 0.00 -> 50.7 mm, vias 0 -> 2
- net /PSFB/OUTP: track 4.39 -> 44.3 mm, vias 0 -> 2
- net /PFC/BST-VSNS: track 0.00 -> 39.7 mm, vias 0 -> 2
- net /IO_SNS: track 0.00 -> 36.1 mm, vias 0 -> 1
- net /PFC/V_RECT_N: track 0.00 -> 28.5 mm
- net Net-(SW1-Pad2): track 0.00 -> 26.9 mm, vias 0 -> 2
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- added copper zone on F.Cu, net /Inputfilter/L_AC
- added copper zone on F.Cu, net /Inputfilter/L_AC_MID
- added copper zone on F.Cu, net /Inputfilter/L_FILT_AC
- added copper zone on F.Cu, net /Inputfilter/N_AC
- added copper zone on F.Cu, net /Inputfilter/N_AC_FUSE
- added copper zone on F.Cu, net /Inputfilter/N_AC_MID
- added copper zone on F.Cu, net /Inputfilter/N_FILT_AC
- added copper zone on F.Cu, net /N_FILT_AC_RT
- added copper zone on F.Cu, net /OUTN
- added copper zone on F.Cu, net /OUTP-DOR
- added copper zone on F.Cu, net /PFC/BST-SW-NODE
- added copper zone on B.Cu, net /PFC/V_RECT_N
- added copper zone on F.Cu, net /PFC/V_RECT_P
- added copper zone on F.Cu, net /PSFB/OUTP
- added copper zone on B.Cu, net /PSFB/SWAB
- added copper zone on F.Cu, net /PSFB/SWAB
- added copper zone on F.Cu, net /PSFB/SWCD
- added copper zone on F.Cu, net /PSFB/SWE
- added copper zone on F.Cu, net /PSFB/SWF
- added copper zone on B.Cu, net /PSFB/SW_LOUT
- added copper zone on F.Cu, net /PSFB/U9-HS
- added copper zone on B.Cu, net /PSFB/VINP
- added copper zone on F.Cu, net /PSFB/VINP
- added copper zone on F.Cu, net /PSFB/VINX
- added copper zone on B.Cu, net /RTNP
- added copper zone on F.Cu, net /RTNP
- added copper zone on F.Cu, net Earth
- added copper zone on B.Cu, net GND
- added copper zone on F.Cu, net GND
- removed copper zone on B.Cu, net (none)
Other:
- board outline added: 343.4 x 81.3 mm
